Commit message: Updated Collision Mesh

File: urdf_template_4/urdf/urdf_template_4.urdf (robot description, URDF)
Before this commit: robot urdf_template_4, 5 links, 4 joints
Links:
- link base_link: geometry collision mesh filename=package://urdf_template_4/meshes/base_link.STL; visual mesh filename=package://urdf_template_4/meshes/base_link.STL
- link link_1: geometry collision mesh filename=package://urdf_template_4/meshes/link_1.STL; visual mesh filename=package://urdf_template_4/meshes/link_1.STL
- link link_2: geometry collision mesh filename=package://urdf_template_4/meshes/link_2.STL; visual mesh filename=package://urdf_template_4/meshes/link_2.STL
- link link_3: geometry collision mesh filename=package://urdf_template_4/meshes/link_3.STL; visual mesh filename=package://urdf_template_4/meshes/link_3.STL
- link link_4: geometry collision mesh filename=package://urdf_template_4/meshes/link_4.STL; visual mesh filename=package://urdf_template_4/meshes/link_4.STL

Commit message: Added Limits To Joints

File: urdf_template_4/urdf/urdf_template_4.urdf (robot description, URDF)
Before this commit: robot urdf_template_4, 5 links, 4 joints
Joints:
- joint Joint_1: limit lower=-6.283 upper=6.283 effort=0 velocity=0 -> lower=0 upper=5.236 effort=0 velocity=0
- joint Joint_2: limit lower=0 upper=0 effort=0 velocity=0 -> lower=0.5411 upper=1.1284 effort=0 velocity=0; type continuous -> revolute
- joint Joint_3: limit lower=0 upper=0 effort=0 velocity=0 -> lower=0 upper=0.7854 effort=0 velocity=0; type continuous -> revolute
- joint Joint_4: limit lower=0 upper=0 effort=0 velocity=0 -> lower=-1.8 upper=2.793 effort=0 velocity=0; type continuous -> revolute

Commit message: Added a fifth joint the URDF and improved README.md

File: urdf_template_4/urdf/urdf_template_4.urdf (robot description, URDF)
Before this commit: robot urdf_template_4, 5 links, 4 joints
Links:
- added link link_5; collision mesh filename=package://urdf_template_4/meshes/link_5.STL; visual mesh filename=package://urdf_template_4/meshes/link_5.STL
Joints:
- added joint Joint_5: type continuous, parent link_4, child link_5, origin xyz=0.0078847 0.21145 -0.20399 rpy=0 0 0, axis -0.0010653 0.72061 -0.69334
- joint Joint_1: origin xyz=0.065007 0.065193 0.063823 rpy=0 0 -3.1416 -> xyz=0.0650066711333143 0.0651925420406113 0.063822562470066 rpy=0 0 -3.14159265249356
- joint Joint_2: axis -0.99764 0.068696 0 -> -0.997637620258692 0.0686962782439793 0; limit lower=0.5411 upper=1.1284 effort=0 velocity=0 -> lower=0.5411 upper=0.1284 effort=0 velocity=0
- joint Joint_3: axis 0.99764 -0.068696 0 -> 0.997637620258692 -0.0686962782439819 0; origin xyz=0.0035291 0.074546 0.35016 rpy=0 0 0 -> xyz=0.00352905769600124 0.0745463768419771 0.350158363506979 rpy=0 0 0
- joint Joint_4: axis 0.99764 -0.068696 0 -> 0.997637620258692 -0.0686962782439826 0; origin xyz=0.025671 0.26163 -0.098739 rpy=0 0 0 -> xyz=0.02567074846148 0.261630460097419 -0.0987385223146501 rpy=0 0 0

Commit message: Improved Joint Limits and Replaced Deprecated Dependency

File: urdf_template_4/urdf/urdf_template_4.urdf (robot description, URDF)
Before this commit: robot urdf_template_4, 6 links, 5 joints
Joints:
- joint Joint_1: limit lower=0 upper=5.236 effort=0 velocity=0 -> lower=-2.618 upper=2.618 effort=0 velocity=0
- joint Joint_2: limit lower=0.5411 upper=0.1284 effort=0 velocity=0 -> lower=1.1284 upper=0.45 effort=0 velocity=0

Commit message: Updated Joint Limits

File: urdf_template_4/urdf/urdf_template_4.urdf (robot description, URDF)
Before this commit: robot urdf_template_4, 6 links, 5 joints
Joints:
- joint Joint_2: limit lower=1.1284 upper=0.45 effort=0 velocity=0 -> lower=1.1284 upper=0.5411 effort=0 velocity=0
